File: macroAll/macroAll.kicad_pcb (KiCad board)
At the start: 2 copper layers, 97 parts, among them SW1 SW_Push, SW10 SW_Push, SW11 SW_Push, SW12 SW_Push, SW13 SW_Push, SW14 SW_Push, SW15 SW_Push, SW16 SW_Push, SW17 SW_Push, SW18 SW_Push, SW19 SW_Push, SW2 SW_Push, SW20 SW_Push, SW21 SW_Push, SW22 SW_Push, SW23 SW_Push, SW24 SW_Push, SW25 SW_Push, SW26 SW_Push, SW27 SW_Push, SW28 SW_Push, SW29 SW_Push, SW3 SW_Push, SW30 SW_Push, SW31 SW_Push, SW32 SW_Push, SW35 SW_Push, SW36 SW_Push, SW37 SW_Push, SW38 SW_Push, SW39 SW_Push, SW4 SW_Push, SW40 SW_Push, SW41 SW_Push, SW42 SW_Push, SW43 SW_Push, SW44 SW_Push, SW5 SW_Push, SW6 SW_Push, SW7 SW_Push, SW8 SW_Push, SW9 SW_Push, U1 XIAO-nRF52840-SMD, U2 XIAO-nRF52840-SMD

Commit message: fixed footprint
Parts:
- removed U1, U2: XIAO-nRF52840-SMD, modifiedOPL:XIAO-nRF52840-SMD
- added D100: D, Diode_SMD:D_SOD-123, F.Cu at (149.3, 12.0)
- added D101: D, Diode_SMD:D_SOD-123, F.Cu at (149.3, 15.4)
- added D102: D, Diode_SMD:D_SOD-123, F.Cu at (149.3, 18.7)
- added D103: D, Diode_SMD:D_SOD-123, F.Cu at (291.6, 35.5)
- added D104: D, Diode_SMD:D_SOD-123, F.Cu at (291.6, 38.8)
- added D105: D, Diode_SMD:D_SOD-123, F.Cu at (297.4, 8.68)
- added D106: D, Diode_SMD:D_SOD-123, F.Cu at (297.4, 12.0)
- added D107: D, Diode_SMD:D_SOD-123, F.Cu at (297.4, 15.4)
- added D108: D, Diode_SMD:D_SOD-123, F.Cu at (297.4, 18.7)
- added D109: D, Diode_SMD:D_SOD-123, F.Cu at (149.3, 22.1)
- added D110: D, Diode_SMD:D_SOD-123, F.Cu at (149.3, 25.4)
- added D111: D, Diode_SMD:D_SOD-123, F.Cu at (149.3, 28.8)
- added D112: D, Diode_SMD:D_SOD-123, F.Cu at (149.3, 32.1)
- added D113: D, Diode_SMD:D_SOD-123, F.Cu at (149.3, 35.5)
- added D114: D, Diode_SMD:D_SOD-123, F.Cu at (149.3, 38.8)
- added D115: D, Diode_SMD:D_SOD-123, F.Cu at (297.4, 22.1)
- added D116: D, Diode_SMD:D_SOD-123, F.Cu at (297.4, 25.4)
- added D117: D, Diode_SMD:D_SOD-123, F.Cu at (297.4, 28.8)
- added D118: D, Diode_SMD:D_SOD-123, F.Cu at (297.4, 32.1)
- added D119: D, Diode_SMD:D_SOD-123, F.Cu at (297.4, 35.5)
- added D120: D, Diode_SMD:D_SOD-123, F.Cu at (297.4, 38.8)
- added D33: D, Diode_SMD:D_SOD-123, F.Cu at (126.2, 28.8)
- added D34: D, Diode_SMD:D_SOD-123, F.Cu at (126.2, 32.1)
- added D45: D, Diode_SMD:D_SOD-123, F.Cu at (132.0, 18.7)
- added D46: D, Diode_SMD:D_SOD-123, F.Cu at (132.0, 22.1)
- added D47: D, Diode_SMD:D_SOD-123, F.Cu at (280.0, 12.0)
- added D48: D, Diode_SMD:D_SOD-123, F.Cu at (280.0, 15.4)
- added D49: D, Diode_SMD:D_SOD-123, F.Cu at (280.0, 18.7)
- added D50: D, Diode_SMD:D_SOD-123, F.Cu at (280.0, 22.1)
- added D51: D, Diode_SMD:D_SOD-123, F.Cu at (132.0, 25.4)
- added D52: D, Diode_SMD:D_SOD-123, F.Cu at (132.0, 28.8)
- added D53: D, Diode_SMD:D_SOD-123, F.Cu at (132.0, 32.1)
- added D54: D, Diode_SMD:D_SOD-123, F.Cu at (132.0, 35.5)
- added D55: D, Diode_SMD:D_SOD-123, F.Cu at (132.0, 38.8)
- added D56: D, Diode_SMD:D_SOD-123, F.Cu at (280.0, 25.4)
- added D57: D, Diode_SMD:D_SOD-123, F.Cu at (280.0, 28.8)
- added D58: D, Diode_SMD:D_SOD-123, F.Cu at (280.0, 32.1)
- added D59: D, Diode_SMD:D_SOD-123, F.Cu at (280.0, 35.5)
- added D60: D, Diode_SMD:D_SOD-123, F.Cu at (280.0, 38.8)
- added D61: D, Diode_SMD:D_SOD-123, F.Cu at (137.8, 8.68)
- added D62: D, Diode_SMD:D_SOD-123, F.Cu at (137.8, 12.0)
- added D63: D, Diode_SMD:D_SOD-123, F.Cu at (137.8, 15.4)
- added D64: D, Diode_SMD:D_SOD-123, F.Cu at (137.8, 18.7)
- added D65: D, Diode_SMD:D_SOD-123, F.Cu at (137.8, 22.1)
- added D66: D, Diode_SMD:D_SOD-123, F.Cu at (137.8, 25.4)
- added D67: D, Diode_SMD:D_SOD-123, F.Cu at (137.8, 28.8)
- added D68: D, Diode_SMD:D_SOD-123, F.Cu at (137.8, 32.1)
- added D69: D, Diode_SMD:D_SOD-123, F.Cu at (137.8, 35.5)
- added D70: D, Diode_SMD:D_SOD-123, F.Cu at (137.8, 38.8)
- added D71: D, Diode_SMD:D_SOD-123, F.Cu at (143.6, 8.68)
- added D72: D, Diode_SMD:D_SOD-123, F.Cu at (143.6, 12.0)
- added D73: D, Diode_SMD:D_SOD-123, F.Cu at (143.6, 15.4)
- added D74: D, Diode_SMD:D_SOD-123, F.Cu at (143.6, 18.7)
- added D75: D, Diode_SMD:D_SOD-123, F.Cu at (143.6, 22.1)
- added D76: D, Diode_SMD:D_SOD-123, F.Cu at (143.6, 25.4)
- added D77: D, Diode_SMD:D_SOD-123, F.Cu at (143.6, 28.8)
- added D78: D, Diode_SMD:D_SOD-123, F.Cu at (143.6, 32.1)
- added D79: D, Diode_SMD:D_SOD-123, F.Cu at (285.8, 8.68)
- added D80: D, Diode_SMD:D_SOD-123, F.Cu at (285.8, 12.0)
- added D81: D, Diode_SMD:D_SOD-123, F.Cu at (285.8, 15.4)
- added D82: D, Diode_SMD:D_SOD-123, F.Cu at (285.8, 18.7)
- added D83: D, Diode_SMD:D_SOD-123, F.Cu at (285.8, 22.1)
- added D84: D, Diode_SMD:D_SOD-123, F.Cu at (285.8, 25.4)
- added D85: D, Diode_SMD:D_SOD-123, F.Cu at (285.8, 28.8)
- added D86: D, Diode_SMD:D_SOD-123, F.Cu at (285.8, 32.1)
- added D87: D, Diode_SMD:D_SOD-123, F.Cu at (285.8, 35.5)
- added D88: D, Diode_SMD:D_SOD-123, F.Cu at (285.8, 38.8)
- added D89: D, Diode_SMD:D_SOD-123, F.Cu at (291.6, 8.68)
- added D90: D, Diode_SMD:D_SOD-123, F.Cu at (291.6, 12.0)
- added D91: D, Diode_SMD:D_SOD-123, F.Cu at (291.6, 15.4)
- added D92: D, Diode_SMD:D_SOD-123, F.Cu at (291.6, 18.7)
- added D93: D, Diode_SMD:D_SOD-123, F.Cu at (291.6, 22.1)
- added D94: D, Diode_SMD:D_SOD-123, F.Cu at (291.6, 25.4)
- added D95: D, Diode_SMD:D_SOD-123, F.Cu at (291.6, 28.8)
- added D96: D, Diode_SMD:D_SOD-123, F.Cu at (291.6, 32.1)
- added D97: D, Diode_SMD:D_SOD-123, F.Cu at (143.6, 35.5)
- added D98: D, Diode_SMD:D_SOD-123, F.Cu at (143.6, 38.8)
- added D99: D, Diode_SMD:D_SOD-123, F.Cu at (149.3, 8.68)
- added H1: MountingHole, MountingHole:MountingHole_2.5mm, F.Cu at (120.7, 43.8)
- added H10: MountingHole, MountingHole:MountingHole_2.5mm, F.Cu at (268.8, 70.0)
- added H2: MountingHole, MountingHole:MountingHole_2.5mm, F.Cu at (268.8, 43.8)
- added H3: MountingHole, MountingHole:MountingHole_2.5mm, F.Cu at (120.7, 50.3)
- added H4: MountingHole, MountingHole:MountingHole_2.5mm, F.Cu at (268.8, 50.3)
- added H5: MountingHole, MountingHole:MountingHole_2.5mm, F.Cu at (120.7, 56.9)
- added H6: MountingHole, MountingHole:MountingHole_2.5mm, F.Cu at (268.8, 56.9)
- added H7: MountingHole, MountingHole:MountingHole_2.5mm, F.Cu at (120.7, 63.4)
- added H8: MountingHole, MountingHole:MountingHole_2.5mm, F.Cu at (268.8, 63.4)
- added H9: MountingHole, MountingHole:MountingHole_2.5mm, F.Cu at (120.7, 70.0)
- added SW100: SW_Push, PCM_Switch_Keyboard_Hotswap_Kailh:SW_Hotswap_Kailh_Choc_V1, F.Cu at (107.2, 33.2)
- added SW101: SW_Push, PCM_Switch_Keyboard_Hotswap_Kailh:SW_Hotswap_Kailh_Choc_V1, F.Cu at (107.2, 50.5)
- added SW102: SW_Push, PCM_Switch_Keyboard_Hotswap_Kailh:SW_Hotswap_Kailh_Choc_V1, F.Cu at (107.2, 67.7)
- added SW103: SW_Push, PCM_Switch_Keyboard_Hotswap_Kailh:SW_Hotswap_Kailh_Choc_V1, F.Cu at (236.7, 154.0)
- added SW104: SW_Push, PCM_Switch_Keyboard_Hotswap_Kailh:SW_Hotswap_Kailh_Choc_V1, F.Cu at (236.7, 171.3)
- added SW105: SW_Push, PCM_Switch_Keyboard_Hotswap_Kailh:SW_Hotswap_Kailh_Choc_V1, F.Cu at (255.2, 16.0)
- added SW106: SW_Push, PCM_Switch_Keyboard_Hotswap_Kailh:SW_Hotswap_Kailh_Choc_V1, F.Cu at (255.2, 33.2)
- added SW107: SW_Push, PCM_Switch_Keyboard_Hotswap_Kailh:SW_Hotswap_Kailh_Choc_V1, F.Cu at (255.2, 50.5)
- added SW108: SW_Push, PCM_Switch_Keyboard_Hotswap_Kailh:SW_Hotswap_Kailh_Choc_V1, F.Cu at (255.2, 67.7)
- added SW109: SW_Push, PCM_Switch_Keyboard_Hotswap_Kailh:SW_Hotswap_Kailh_Choc_V1, F.Cu at (107.2, 85.0)
- added SW110: SW_Push, PCM_Switch_Keyboard_Hotswap_Kailh:SW_Hotswap_Kailh_Choc_V1, F.Cu at (107.2, 102.2)
- added SW111: SW_Push, PCM_Switch_Keyboard_Hotswap_Kailh:SW_Hotswap_Kailh_Choc_V1, F.Cu at (107.2, 119.5)
- added SW112: SW_Push, PCM_Switch_Keyboard_Hotswap_Kailh:SW_Hotswap_Kailh_Choc_V1, F.Cu at (107.2, 136.7)
- added SW113: SW_Push, PCM_Switch_Keyboard_Hotswap_Kailh:SW_Hotswap_Kailh_Choc_V1, F.Cu at (107.2, 154.0)
- added SW114: SW_Push, PCM_Switch_Keyboard_Hotswap_Kailh:SW_Hotswap_Kailh_Choc_V1, F.Cu at (107.2, 171.3)
- added SW115: SW_Push, PCM_Switch_Keyboard_Hotswap_Kailh:SW_Hotswap_Kailh_Choc_V1, F.Cu at (255.2, 85.0)
- added SW116: SW_Push, PCM_Switch_Keyboard_Hotswap_Kailh:SW_Hotswap_Kailh_Choc_V1, F.Cu at (255.2, 102.2)
- added SW117: SW_Push, PCM_Switch_Keyboard_Hotswap_Kailh:SW_Hotswap_Kailh_Choc_V1, F.Cu at (255.2, 119.5)
- added SW118: SW_Push, PCM_Switch_Keyboard_Hotswap_Kailh:SW_Hotswap_Kailh_Choc_V1, F.Cu at (255.2, 136.7)
- added SW119: SW_Push, PCM_Switch_Keyboard_Hotswap_Kailh:SW_Hotswap_Kailh_Choc_V1, F.Cu at (255.2, 154.0)
- added SW120: SW_Push, PCM_Switch_Keyboard_Hotswap_Kailh:SW_Hotswap_Kailh_Choc_V1, F.Cu at (255.2, 171.3)
- added SW33: SW_Push, PCM_Switch_Keyboard_Hotswap_Kailh:SW_Hotswap_Kailh_Choc_V1, F.Cu at (33.0, 119.5)
- added SW34: SW_Push, PCM_Switch_Keyboard_Hotswap_Kailh:SW_Hotswap_Kailh_Choc_V1, F.Cu at (33.0, 136.7)
- added SW45: SW_Push, PCM_Switch_Keyboard_Hotswap_Kailh:SW_Hotswap_Kailh_Choc_V1, F.Cu at (51.5, 67.7)
- added SW46: SW_Push, PCM_Switch_Keyboard_Hotswap_Kailh:SW_Hotswap_Kailh_Choc_V1, F.Cu at (51.5, 85.0)
- added SW47: SW_Push, PCM_Switch_Keyboard_Hotswap_Kailh:SW_Hotswap_Kailh_Choc_V1, F.Cu at (199.6, 33.2)
- added SW48: SW_Push, PCM_Switch_Keyboard_Hotswap_Kailh:SW_Hotswap_Kailh_Choc_V1, F.Cu at (199.6, 50.5)
- added SW49: SW_Push, PCM_Switch_Keyboard_Hotswap_Kailh:SW_Hotswap_Kailh_Choc_V1, F.Cu at (199.6, 67.7)
- added SW50: SW_Push, PCM_Switch_Keyboard_Hotswap_Kailh:SW_Hotswap_Kailh_Choc_V1, F.Cu at (199.6, 85.0)
- added SW51: SW_Push, PCM_Switch_Keyboard_Hotswap_Kailh:SW_Hotswap_Kailh_Choc_V1, F.Cu at (51.5, 102.2)
- added SW52: SW_Push, PCM_Switch_Keyboard_Hotswap_Kailh:SW_Hotswap_Kailh_Choc_V1, F.Cu at (51.5, 119.5)
- added SW53: SW_Push, PCM_Switch_Keyboard_Hotswap_Kailh:SW_Hotswap_Kailh_Choc_V1, F.Cu at (51.5, 136.7)
- added SW54: SW_Push, PCM_Switch_Keyboard_Hotswap_Kailh:SW_Hotswap_Kailh_Choc_V1, F.Cu at (51.5, 154.0)
- added SW55: SW_Push, PCM_Switch_Keyboard_Hotswap_Kailh:SW_Hotswap_Kailh_Choc_V1, F.Cu at (51.5, 171.3)
- added SW56: SW_Push, PCM_Switch_Keyboard_Hotswap_Kailh:SW_Hotswap_Kailh_Choc_V1, F.Cu at (199.6, 102.2)
- added SW57: SW_Push, PCM_Switch_Keyboard_Hotswap_Kailh:SW_Hotswap_Kailh_Choc_V1, F.Cu at (199.6, 119.5)
- added SW58: SW_Push, PCM_Switch_Keyboard_Hotswap_Kailh:SW_Hotswap_Kailh_Choc_V1, F.Cu at (199.6, 136.7)
- added SW59: SW_Push, PCM_Switch_Keyboard_Hotswap_Kailh:SW_Hotswap_Kailh_Choc_V1, F.Cu at (199.6, 154.0)
- added SW60: SW_Push, PCM_Switch_Keyboard_Hotswap_Kailh:SW_Hotswap_Kailh_Choc_V1, F.Cu at (199.6, 171.3)
- added SW61: SW_Push, PCM_Switch_Keyboard_Hotswap_Kailh:SW_Hotswap_Kailh_Choc_V1, F.Cu at (70.1, 16.0)
- added SW62: SW_Push, PCM_Switch_Keyboard_Hotswap_Kailh:SW_Hotswap_Kailh_Choc_V1, F.Cu at (70.1, 33.2)
- added SW63: SW_Push, PCM_Switch_Keyboard_Hotswap_Kailh:SW_Hotswap_Kailh_Choc_V1, F.Cu at (70.1, 50.5)
- added SW64: SW_Push, PCM_Switch_Keyboard_Hotswap_Kailh:SW_Hotswap_Kailh_Choc_V1, F.Cu at (70.1, 67.7)
- added SW65: SW_Push, PCM_Switch_Keyboard_Hotswap_Kailh:SW_Hotswap_Kailh_Choc_V1, F.Cu at (70.1, 85.0)
- added SW66: SW_Push, PCM_Switch_Keyboard_Hotswap_Kailh:SW_Hotswap_Kailh_Choc_V1, F.Cu at (70.1, 102.2)
- added SW67: SW_Push, PCM_Switch_Keyboard_Hotswap_Kailh:SW_Hotswap_Kailh_Choc_V1, F.Cu at (70.1, 119.5)
- added SW68: SW_Push, PCM_Switch_Keyboard_Hotswap_Kailh:SW_Hotswap_Kailh_Choc_V1, F.Cu at (70.1, 136.7)
- added SW69: SW_Push, PCM_Switch_Keyboard_Hotswap_Kailh:SW_Hotswap_Kailh_Choc_V1, F.Cu at (70.1, 154.0)
- added SW70: SW_Push, PCM_Switch_Keyboard_Hotswap_Kailh:SW_Hotswap_Kailh_Choc_V1, F.Cu at (70.1, 171.3)
- added SW71: SW_Push, PCM_Switch_Keyboard_Hotswap_Kailh:SW_Hotswap_Kailh_Choc_V1, F.Cu at (88.6, 16.0)
- added SW72: SW_Push, PCM_Switch_Keyboard_Hotswap_Kailh:SW_Hotswap_Kailh_Choc_V1, F.Cu at (88.6, 33.2)
- added SW73: SW_Push, PCM_Switch_Keyboard_Hotswap_Kailh:SW_Hotswap_Kailh_Choc_V1, F.Cu at (88.6, 50.5)
- added SW74: SW_Push, PCM_Switch_Keyboard_Hotswap_Kailh:SW_Hotswap_Kailh_Choc_V1, F.Cu at (88.6, 67.7)
- added SW75: SW_Push, PCM_Switch_Keyboard_Hotswap_Kailh:SW_Hotswap_Kailh_Choc_V1, F.Cu at (88.6, 85.0)
- added SW76: SW_Push, PCM_Switch_Keyboard_Hotswap_Kailh:SW_Hotswap_Kailh_Choc_V1, F.Cu at (88.6, 102.2)
- added SW77: SW_Push, PCM_Switch_Keyboard_Hotswap_Kailh:SW_Hotswap_Kailh_Choc_V1, F.Cu at (88.6, 119.5)
- added SW78: SW_Push, PCM_Switch_Keyboard_Hotswap_Kailh:SW_Hotswap_Kailh_Choc_V1, F.Cu at (88.6, 136.7)
- added SW79: SW_Push, PCM_Switch_Keyboard_Hotswap_Kailh:SW_Hotswap_Kailh_Choc_V1, F.Cu at (218.2, 16.0)
- added SW80: SW_Push, PCM_Switch_Keyboard_Hotswap_Kailh:SW_Hotswap_Kailh_Choc_V1, F.Cu at (218.2, 33.2)
- added SW81: SW_Push, PCM_Switch_Keyboard_Hotswap_Kailh:SW_Hotswap_Kailh_Choc_V1, F.Cu at (218.2, 50.5)
- added SW82: SW_Push, PCM_Switch_Keyboard_Hotswap_Kailh:SW_Hotswap_Kailh_Choc_V1, F.Cu at (218.2, 67.7)
- added SW83: SW_Push, PCM_Switch_Keyboard_Hotswap_Kailh:SW_Hotswap_Kailh_Choc_V1, F.Cu at (218.2, 85.0)
- added SW84: SW_Push, PCM_Switch_Keyboard_Hotswap_Kailh:SW_Hotswap_Kailh_Choc_V1, F.Cu at (218.2, 102.2)
- added SW85: SW_Push, PCM_Switch_Keyboard_Hotswap_Kailh:SW_Hotswap_Kailh_Choc_V1, F.Cu at (218.2, 119.5)
- added SW86: SW_Push, PCM_Switch_Keyboard_Hotswap_Kailh:SW_Hotswap_Kailh_Choc_V1, F.Cu at (218.2, 136.7)
- added SW87: SW_Push, PCM_Switch_Keyboard_Hotswap_Kailh:SW_Hotswap_Kailh_Choc_V1, F.Cu at (218.2, 154.0)
- added SW88: SW_Push, PCM_Switch_Keyboard_Hotswap_Kailh:SW_Hotswap_Kailh_Choc_V1, F.Cu at (218.2, 171.3)
- added SW89: SW_Push, PCM_Switch_Keyboard_Hotswap_Kailh:SW_Hotswap_Kailh_Choc_V1, F.Cu at (236.7, 16.0)
- added SW90: SW_Push, PCM_Switch_Keyboard_Hotswap_Kailh:SW_Hotswap_Kailh_Choc_V1, F.Cu at (236.7, 33.2)
- added SW91: SW_Push, PCM_Switch_Keyboard_Hotswap_Kailh:SW_Hotswap_Kailh_Choc_V1, F.Cu at (236.7, 50.5)
- added SW92: SW_Push, PCM_Switch_Keyboard_Hotswap_Kailh:SW_Hotswap_Kailh_Choc_V1, F.Cu at (236.7, 67.7)
- added SW93: SW_Push, PCM_Switch_Keyboard_Hotswap_Kailh:SW_Hotswap_Kailh_Choc_V1, F.Cu at (236.7, 85.0)
- added SW94: SW_Push, PCM_Switch_Keyboard_Hotswap_Kailh:SW_Hotswap_Kailh_Choc_V1, F.Cu at (236.7, 102.2)
- added SW95: SW_Push, PCM_Switch_Keyboard_Hotswap_Kailh:SW_Hotswap_Kailh_Choc_V1, F.Cu at (236.7, 119.5)
- added SW96: SW_Push, PCM_Switch_Keyboard_Hotswap_Kailh:SW_Hotswap_Kailh_Choc_V1, F.Cu at (236.7, 136.7)
- added SW97: SW_Push, PCM_Switch_Keyboard_Hotswap_Kailh:SW_Hotswap_Kailh_Choc_V1, F.Cu at (88.6, 154.0)
- added SW98: SW_Push, PCM_Switch_Keyboard_Hotswap_Kailh:SW_Hotswap_Kailh_Choc_V1, F.Cu at (88.6, 171.3)
- added SW99: SW_Push, PCM_Switch_Keyboard_Hotswap_Kailh:SW_Hotswap_Kailh_Choc_V1, F.Cu at (107.2, 16.0)
- added U22: XIAO-nRF52840-Plus-SMD, OPL:XIAO-nRF52840-Plus-SMD, F.Cu at (135.0, 50.6)
- added U23: XIAO-nRF52840-Plus-SMD, OPL:XIAO-nRF52840-Plus-SMD, F.Cu at (283.0, 50.6)
- moved SW43 114.4 mm to (181.1, 171.3)
- moved SW42 114.4 mm to (181.1, 154.0)
- moved SW20 106.8 mm to (33.0, 33.2)
- moved SW19 106.8 mm to (33.0, 16.0)
- moved SW18 99.1 mm to (14.4, 171.3)
- moved SW11 99.1 mm to (14.4, 119.5)
- moved SW12 99.1 mm to (14.4, 136.7)
- moved SW17 99.1 mm to (14.4, 154.0)
- moved SW24 97.0 mm to (181.1, 33.2)
- moved SW23 97.0 mm to (181.1, 16.0)
- moved TP2 86.2 mm to (297.7, 42.5)
- moved TP4 86.2 mm to (297.7, 46.6)
- moved R4 78.7 mm to (297.9, 53.0)
- moved R2 78.7 mm to (297.9, 50.1)
- moved SW22 76.7 mm to (162.5, 171.3)
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
Commit message: half of half keyboard layout finished
Parts:
- moved SW36 331.8 mm to (-146.7, -107.7), turned to 45 degrees
- moved U22 300.5 mm to (-97.8, -139.4), turned to 90 degrees
- moved D76 299.6 mm to (-132.2, -91.7), turned to 45 degrees
- moved R1 299.2 mm to (-106.2, -104.8)
- moved TP1 298.8 mm to (-104.8, -114.3)
- moved SW76 298.7 mm to (-134.9, -95.9), turned to 45 degrees
- moved H3 297.9 mm to (-111.9, -135.7)
- moved TP3 295.0 mm to (-97.6, -114.3)
- moved R3 294.7 mm to (-99.1, -104.8)
- moved SW77 293.7 mm to (-123.1, -84.1), turned to 45 degrees
- moved SW65 291.7 mm to (-160.1, -94.2), turned to 45 degrees
- moved H1 289.5 mm to (-154.8, -45.2)
- moved SW78 289.3 mm to (-111.3, -72.3), turned to 45 degrees
- moved SW66 286.0 mm to (-148.3, -82.4), turned to 45 degrees
- moved SW97 285.3 mm to (-99.5, -60.5), turned to 45 degrees
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
Commit message: left side placement
Parts:
- moved D27 162.1 mm to (33.3, -135.7)
- moved D9 155.0 mm to (14.3, -135.7)
- moved D36 145.9 mm to (-142.9, -104.8), turned to 45 degrees
- moved D28 141.7 mm to (-185.7, -61.9), turned to 45 degrees
- moved D46 139.2 mm to (-170.2, -77.4), turned to 45 degrees
- moved D65 139.0 mm to (-156.0, -91.7), turned to 45 degrees
- moved D66 127.1 mm to (-145.3, -79.8), turned to 45 degrees
- moved D51 125.0 mm to (-159.5, -64.3), turned to 45 degrees
- moved D10 120.6 mm to (-173.8, -50.0), turned to 45 degrees
- moved D77 116.7 mm to (-120.2, -79.8), turned to 45 degrees
- moved D67 111.7 mm to (-133.3, -66.7), turned to 45 degrees
- moved D52 110.3 mm to (-147.6, -52.4), turned to 45 degrees
- moved D11 107.8 mm to (-163.1, -39.3), turned to 45 degrees
- moved D78 103.3 mm to (-108.3, -67.9), turned to 45 degrees
- moved D68 97.0 mm to (-121.4, -54.8), turned to 45 degrees
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Other:
- board outline added: 260.7 x 166.7 mm

Commit message: placed left components, redid left edgecut design, led placement
Parts:
- removed D112, D114: D, Diode_SMD:D_SOD-123
- removed SW112, SW114: SW_Push, PCM_Switch_Keyboard_Hotswap_Kailh:SW_Hotswap_Kailh_Choc_V1
- moved R3 31.8 mm to (-117.2, -131.0)
- moved R1 31.8 mm to (-124.4, -131.0)
- moved TP3 31.8 mm to (-115.8, -140.5)
- moved TP1 31.8 mm to (-122.9, -140.5)
- moved D69 12.5 mm to (-105.8, -53.1), turned to 135 degrees
- moved D53 12.3 mm to (-131.0, -51.9), turned to 135 degrees
- moved D70 12.3 mm to (-94.4, -41.9), turned to 135 degrees
- moved D51 12.3 mm to (-154.8, -75.6), turned to 135 degrees
- moved D55 11.8 mm to (-108.0, -28.5), turned to 135 degrees
- moved D52 11.8 mm to (-143.1, -63.3), turned to 135 degrees
- moved D54 11.7 mm to (-118.8, -39.8), turned to 135 degrees
- moved D76 11.6 mm to (-127.8, -102.4), turned to 135 degrees
- moved D77 11.5 mm to (-115.7, -90.3), turned to 135 degrees
- moved D98 11.2 mm to (-79.6, -54.7), turned to 135 degrees
- moved D78 11.2 mm to (-104.2, -78.3), turned to 135 degrees
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Other:
- outline, holes or cut-outs redrawn
